File: t-dsp_dual_preamp_2.kicad_sch (KiCad schematic)
At the start: 59 parts, among them IC1 1583N16-U, IC2 1583N16-U, IC4 5173N24-U, IC5 5173N24-U, J1 XLRM_NC3FAH, J2 XLRM_NC3FAH, J3 NC3FAH2-0, J4 NC3FAH2-0, J5 Conn_02x05_Odd_Even, Q1 IRF9540N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

Commit message: update
Parts:
- removed U1: PGA2505IDB, project_fp:PGA2505IDB, symbol PGA2505IDB:PGA2505IDB
- C1, C10, C11, C12, C13, C14, C15, C16, C2, C3, C4, C5, C6, C7, C8, C9, CT1, RT1: footprint Capacitor_SMD:C_0805_2012Metric_Pad1.18x1.45mm_HandSolder -> (none)
- D1, D2, D3, D4: footprint Diode_SMD:D_SMA_Handsoldering -> (none)
- R1, R18, R2, R3, R4, R5, R6, R7, R8: footprint Resistor_SMD:R_0805_2012Metric_Pad1.20x1.40mm_HandSolder -> (none)
- board_outline3: footprint project_fp:audio_project_board_outline_100x70 -> project_fp:audio_project_board_outline_100x60
