File: t-dsp_dual_preamp.kicad_sch (KiCad schematic)
At the start: 59 parts, among them IC1 1583N16-U, IC2 1583N16-U, IC4 5173N24-U, IC5 5173N24-U, J1 XLRM_NC3FAH, J2 XLRM_NC3FAH, J3 NC3FAH2-0, J4 NC3FAH2-0, J5 Conn_02x05_Odd_Even, Q1 IRF9540N, Q2 IRF9540N, T108 Tab, T109 Tab, T110 Tab, T111 Tab, U1 PGA2505IDB, U5 SC18IS606PWJ

Commit message: update
Parts:
- removed C14, C15, C16: 100N, Capacitor_SMD:C_0805_2012Metric_Pad1.18x1.45mm_HandSolder, symbol Device:C_Small
- removed C4, C5: 47u, Capacitor_SMD:C_0805_2012Metric_Pad1.18x1.45mm_HandSolder, symbol Device:C_Polarized_Small
- removed CT1: X, Capacitor_SMD:C_0805_2012Metric_Pad1.18x1.45mm_HandSolder, symbol Device:C_Small
- removed D2, D3, D4: S1DB, Diode_SMD:D_SMA_Handsoldering, symbol Device:D_Small_Filled
- removed IC1, IC2: 1583N16-U, QFN65P400X400X95-17N-D, symbol 1583N16-U:1583N16-U
- removed IC4, IC5: 5173N24-U, QFN65P500X500X95-25N-D, symbol 5173N24-U:5173N24-U
- removed J3, J4: NC3FAH2-0, Connector_Audio:Jack_XLR_Neutrik_NC3FAH2-0_Horizontal, symbol Connector_Audio:NC3FAH2-0
- removed Q1, Q2: IRF9540N, Package_TO_SOT_THT:TO-220-3_Vertical, symbol Transistor_FET:IRF9540N
- removed R1, R2: 1k2, Resistor_SMD:R_0805_2012Metric_Pad1.20x1.40mm_HandSolder, symbol Device:R_Small
- removed R18: 47K, Resistor_SMD:R_0805_2012Metric_Pad1.20x1.40mm_HandSolder, symbol Device:R_Small
- removed R3: 10, Resistor_SMD:R_0805_2012Metric_Pad1.20x1.40mm_HandSolder, symbol Device:R_Small
- removed RT1: X, Capacitor_SMD:C_0805_2012Metric_Pad1.18x1.45mm_HandSolder, symbol Device:R_Small
- added C15: 47uF, Capacitor_SMD:C_1206_3216Metric_Pad1.33x1.80mm_HandSolder, symbol Device:C_Polarized_Small
- added C16, C17, C18, C26, C27: 4.7uF, Capacitor_SMD:C_1206_3216Metric_Pad1.33x1.80mm_HandSolder, symbol Device:C_Polarized_Small
- added C19, C20: 47uF, Capacitor_SMD:CP_Elec_8x10.5, symbol Device:C_Polarized_Small
- added C21, C22: 1000pf, Capacitor_SMD:C_0805_2012Metric_Pad1.18x1.45mm_HandSolder, symbol Device:C_Small
- added C4, C5: 0.1uF, Capacitor_SMD:C_0805_2012Metric_Pad1.18x1.45mm_HandSolder, symbol Device:C_Small
- added CC1, CC2: 0, project_fp:R_0805_2012Metric_Pad1.15x1.40mm_HandSolder, symbol Device:C_Small
- added D11: S1DB, Diode_SMD:D_SMA_Handsoldering, symbol Device:D_Small_Filled
- added D6, D7, D8, D9: ~, Diode_SMD:D_SMA_Handsoldering, symbol Device:D_Small_Filled
- added J6: Conn_01x02, symbol Connector_Generic:Conn_01x02
- added J7: Conn_01x06, symbol Connector_Generic:Conn_01x06
- added JMP10, JMP11, R10, R11, R14 (x2), R15 (x2): 0, project_fp:R_0805_2012Metric_Pad1.15x1.40mm_HandSolder, symbol Device:R_Small
- added R10000, R100000, R9: 10, project_fp:R_0805_2012Metric_Pad1.15x1.40mm_HandSolder, symbol Device:R_Small
- added R12: 0, symbol Device:R_Small
- added R16 (x2), R17 (x2): 6.81k, project_fp:R_0805_2012Metric_Pad1.15x1.40mm_HandSolder, symbol Device:R_Small
- C1, C2: value 22p -> 0.1uF
- C10: value 100p -> 1000pf
- C11, C6, C7: value 100p -> 0.1uF
- C12, C13: value 22u NP -> 0.1uF
- C3, C8: value 220p -> 0.1uF
- C9: value 100n -> 0.1uF
- D6: renamed from D1; value S1DB -> ~
- J5: now not fitted; now left out of the parts list
- R4: value 10 -> R_Small; footprint Resistor_SMD:R_0805_2012Metric_Pad1.20x1.40mm_HandSolder -> (none); now not fitted; now left out of the parts list
- R5, R6: value 6k81 -> N/C; footprint Resistor_SMD:R_0805_2012Metric_Pad1.20x1.40mm_HandSolder -> (none); now not fitted; now left out of the parts list
- R7, R8: value 1M2 -> 10; footprint Resistor_SMD:R_0805_2012Metric_Pad1.20x1.40mm_HandSolder -> project_fp:R_0805_2012Metric_Pad1.15x1.40mm_HandSolder
- U1: footprint project_fp:PGA2505IDB -> DB24
Connections:
- net +48V: no longer R5.2, R6.2
- net at C7.2: now also U1.19 (CS21)
- net GNDPWR: now reaches C1.2
- net GNDPWR: now also C10.2, C3.2, J6.2 (Pin_2), J7.2 (Pin_2)
- net at R7.2: now also D6.2 (A), D7.1 (K), R10.1; no longer C12.1
- net -VA: now reaches C12.2
- net -VA: now also C11.2, U1.13 (VA-), U1.17 (VA-), C16.2, C27.2, C4.2, J7.6 (Pin_6), R9.1
- net Earth: now reaches U1.1 (AGND)
- net Earth: now also C11.1, C12.1, C3.1, C8.1, C9.1, C16.1, C17.2, C26.2, C27.1, C4.1, C5.1, D11.1 (K), D6.2 (A), J7.3 (Pin_3), JMP10.1, R12.1, R15.1
- net SCLK: now reaches U1.10 (SCLK)
- net SDO: now reaches U1.11 (SDO)
- net at U1.12 (VD-): now also C13.2, C18.2, R9.2
- net at U1.14 (VOUT-): now also R17.2
- net at U1.15 (VOUT+): now also R16.2
- net +VA: now reaches U1.16 (VA+)
- net +VA: now also C9.2, C17.1, C26.1, C5.2, J7.5 (Pin_5)
- net at U1.18 (CS22): now also C7.1
- net GPO1: now reaches U1.2 (GPO1)
- net at U1.20 (CS12): now also C6.1
- net at U1.21 (CS11): now also C6.2
- net at U1.22 (VCOMIN): now also R14.2, R15.2
- net at U1.23 (VIN-): now also CC2.1
- net at U1.24 (VIN+): now also CC1.1
- net GPO2: now reaches U1.3 (GPO2)
- net GPO3: now reaches U1.4 (GPO3)
- net GPO4: now reaches U1.5 (GPO4)
- net OVR: now reaches U1.6 (OVR)
- net GND: now reaches U1.7 (DGND)
- net GND: now also C13.1, C2.2, R48.1, R49.1, R50.1, R51.1, board_outline1.10 (GNDD), board_outline1.12 (GNDD), board_outline1.14 (GNDD), board_outline1.16 (GNDD), board_outline1.18 (GNDD), board_outline1.20 (GNDD), board_outline1.22 (AGND), board_outline1.24 (AGND), board_outline1.26 (AGND), board_outline1.28 (AGND), board_outline1.30 (AGND), board_outline1.32 (AGND), board_outline1.34 (AGND), board_outline1.36 (AGND), board_outline1.47 (GNDD), board_outline1.51 (DGND), board_outline1.52 (DGND), board_outline1.6 (GNDD), board_outline1.8 (GNDD), C15.2, C18.1, JMP10.2, JMP11.2
- net SDI: now reaches U1.8 (SDI)
- net CS: now reaches U1.9 (*CS)
- net VIN1-: now reaches R4.1
- net VIN1-: now also C22.1, R100000.1, R17.1
- net at R8.2: now also D8.2 (A), D9.1 (K), R11.1; no longer C13.1
- removed net +15V: C11.1, C9.1, D6.1 (K)
- net -15V: no longer names the net of C10.1
- net -15V: now also C21.1, C22.2; no longer C11.2
- removed net AGND: C7.1, C8.2, R4.2, R48.1, R49.1, R50.1, R51.1, R7.1, board_outline1.10 (GNDD), board_outline1.12 (GNDD), board_outline1.14 (GNDD), board_outline1.16 (GNDD), board_outline1.18 (GNDD), board_outline1.20 (GNDD), board_outline1.22 (AGND), board_outline1.24 (AGND), board_outline1.26 (AGND), board_outline1.28 (AGND), board_outline1.30 (AGND), board_outline1.32 (AGND), board_outline1.34 (AGND), board_outline1.36 (AGND), board_outline1.47 (GNDD), board_outline1.51 (DGND), board_outline1.52 (DGND), board_outline1.6 (GNDD), board_outline1.8 (GNDD)
- removed net GNDREF: C10.2, C9.2
- removed net IN+: C1.1, C3.1, R5.1
- removed net IN-: C2.1, C3.2, R6.1
- new net: R10.2, R14.1, R5.2
- new net: CC1.2, R14.2
- new net: C8.2, J7.4 (Pin_4), R14.1
- new net: R11.2, R15.2, R6.1
- new net: R12.2, R5.1, R6.2
- new net: C20.1, R100000.2
- new net: C19.1, R10000.2
- new net: C19.2, R7.1
- new net: CC2.2, R15.1
- new net: C20.2, R8.1
- new net +48v: C1.1, J6.1 (Pin_1), R16.1, R17.2
- new net +5VA: D6.1 (K), D6.1 (K), D8.1 (K)
- new net -5VA: D11.2 (A), D7.2 (A), D9.2 (A)
- new net SHIELD: JMP11.1
- new net VCC: C15.1, C2.1, J7.1 (Pin_1)
- new net VIO1+: C21.2, R10000.1, R16.2, R4.2
- new net VOUT+: R16.1
- new net VOUT-: R17.1
- no-connect marks 5 -> 4
Other:
- note removed: "AUDIO PREAMPS"
- note removed: "DIGITAL CONTROL"
- moved on the sheet: D6

Commit message: update
Parts:
- CC1, CC2, JMP10, JMP11, R10, R10000, R100000, R11, R14, R15, R16, R17, R7, R8, R9: footprint project_fp:R_0805_2012Metric_Pad1.15x1.40mm_HandSolder -> project_fp:R_0805_2012Metric_Pad1.20x1.40mm_HandSolder
- J3: renamed from R14; footprint project_fp:R_0805_2012Metric_Pad1.15x1.40mm_HandSolder -> project_fp:R_0805_2012Metric_Pad1.20x1.40mm_HandSolder
- J4: renamed from R15; footprint project_fp:R_0805_2012Metric_Pad1.15x1.40mm_HandSolder -> project_fp:R_0805_2012Metric_Pad1.20x1.40mm_HandSolder
- J6: footprint (none) -> Connector_PinHeader_2.54mm:PinHeader_1x02_P2.54mm_Vertical
- J8: renamed from R12; footprint (none) -> project_fp:R_0805_2012Metric_Pad1.20x1.40mm_HandSolder
- J96: renamed from R51; footprint project_fp:R_0805_2012Metric_Pad1.15x1.40mm_HandSolder -> project_fp:R_0805_2012Metric_Pad1.20x1.40mm_HandSolder
- J97: renamed from R50; footprint project_fp:R_0805_2012Metric_Pad1.15x1.40mm_HandSolder -> project_fp:R_0805_2012Metric_Pad1.20x1.40mm_HandSolder
- J98: renamed from R49; footprint project_fp:R_0805_2012Metric_Pad1.15x1.40mm_HandSolder -> project_fp:R_0805_2012Metric_Pad1.20x1.40mm_HandSolder
- J99: renamed from R48; footprint project_fp:R_0805_2012Metric_Pad1.15x1.40mm_HandSolder -> project_fp:R_0805_2012Metric_Pad1.20x1.40mm_HandSolder
- R12: renamed from R16; value 6.81k -> 0 ohm; footprint project_fp:R_0805_2012Metric_Pad1.15x1.40mm_HandSolder -> project_fp:R_0805_2012Metric_Pad1.20x1.40mm_HandSolder
- R13: renamed from R17; value 6.81k -> 0 ohm; footprint project_fp:R_0805_2012Metric_Pad1.15x1.40mm_HandSolder -> project_fp:R_0805_2012Metric_Pad1.20x1.40mm_HandSolder
- R4, R5, R6: footprint (none) -> project_fp:R_0805_2012Metric_Pad1.20x1.40mm_HandSolder
- renumbered D6 to D10
Connections:
- net VIO1+ renamed VIN1+
Other:
- moved on the sheet: J1
