File: t-dsp_dual_preamp.kicad_sch (KiCad schematic)
At the start: 15 parts, among them J1 XLRM_NC3MAH, J10 COMBO_NCJ6FA-H, J2 XLRM_NC3MAH, J7 Conn_01x06, J9 COMBO_NCJ6FA-H, T108 Tab, T109 Tab, T110 Tab, T111 Tab

Commit message: update
Parts:
- removed J7: Conn_01x06, symbol Connector_Generic:Conn_01x06
- added C6, C8: 470uF Tantalum, Capacitor_Tantalum_SMD:CP_EIA-7343-15_Kemet-W_HandSolder, symbol Device:C_Polarized
- added C7, C9: 470 uF Electrolytic Audio-Grade, project_fp:CP_Radial_D10.0mm_P5.00mm_AND_D8.0mm_P3.5mm, symbol Device:C_Polarized
- added J11, J8: B2B-XH-A, project_fp:JST_B2B-XH-A, symbol JST_B2B-XH-A:B2B-XH-A
- added J3, J4: Conn_01x02, Connector_JST:JST_XH_B2B-XH-AM_1x02_P2.50mm_Vertical, symbol Connector_Generic:Conn_01x02
- added J5: Conn_02x08_Odd_Even, Connector_IDC:IDC-Header_2x07_P2.54mm_Vertical, symbol Connector_Generic:Conn_02x08_Odd_Even
- added J6, J7: Conn_02x03_Odd_Even, project_fp:PREAMP_BYPASS_IDC-Header_2x03_P2.54mm_Vertical, symbol Connector_Generic:Conn_02x03_Odd_Even
- board_outline3: footprint project_fp:audio_project_board_outline_100x80 -> project_fp:audio_project_board_outline_100x50_minus2mounts
Connections:
- net AUDIO_IN1P: now also J5.1 (Pin_1), J6.1 (Pin_1)
- net AUDIO_IN2P: now also J5.9 (Pin_9), J7.1 (Pin_1)
- net G: now also J5.11 (Pin_11), J5.12 (Pin_12), J5.15 (Pin_15), J5.16 (Pin_16), J5.3 (Pin_3), J5.4 (Pin_4), J5.7 (Pin_7), J5.8 (Pin_8), J6.3 (Pin_3), J6.4 (Pin_4), J7.3 (Pin_3), J7.4 (Pin_4)
- net AUDIO_OUT1M: now reaches board_outline1.23 (OUT1M)
- net AUDIO_OUT2M: now reaches board_outline1.27 (OUT2M)
- net AUDIO_IN1M: now reaches board_outline1.31 (IN1M)
- net AUDIO_IN1M: now also J5.5 (Pin_5), J6.5 (Pin_5)
- net AUDIO_IN2M: now reaches board_outline1.35 (IN2M)
- net AUDIO_IN2M: now also J5.13 (Pin_13), J7.5 (Pin_5)
- net AUDIO_OUTP renamed AUDIO_OUT1P
- new net: C8.2, C9.2
- new net AUDIO_IN1M+: J5.6 (Pin_6), J6.6 (Pin_6)
- new net AUDIO_IN1P+: J5.2 (Pin_2), J6.2 (Pin_2)
- new net AUDIO_IN2M+: J5.14 (Pin_14), J7.6 (Pin_6)
- new net AUDIO_IN2P+: J5.10 (Pin_10), J7.2 (Pin_2)
- no-connect marks 4 -> 0
Other:
- note added: "MIC PREAMP MEZZANINE"
- note added: "PHANTOM POWER INPUTS"
- note added: "T-DSP BALANCED AUDIO IO"
- note added: "TABS"
- note added: "XLR + 1/4" COMBO INPUTS"
- note added: "XLR MALE OUT"
- note removed: "I2C TO SPI BRIDGE"
- note removed: "POWER INPUT AND DISTRIBUTION"
- note removed: "T-DSP AUDIO I/O MODULE"
- moved on the sheet: H1, H2, H3, H4, J1, J10A, J10B, J2, J9A, J9B, T108, T109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

Commit message: update
Parts:
- board_outline3: footprint project_fp:audio_project_board_outline_100x50_minus2mounts -> project_fp:audio_project_board_outline_100x50_minus4mounts
Changed lines of the file:
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@@
 			)
 		)
-		(property "Footprint" "project_fp:audio_project_board_outline_100x50_minus2mounts"
+		(property "Footprint" "project_fp:audio_project_board_outline_100x50_minus4mounts"
 			(at 293.37 1036.066 0)
 			(effects
