File: t-dsp_dual_preamp.kicad_pcb (KiCad board)
At the start: 2 copper layers, 100 x 70 mm, 14 parts, among them IC1 1583N16-U, IC2 1583N16-U, IC4 5173N24-U, IC5 5173N24-U, J1 XLRM_NC3FAH, J2 XLRM_NC3FAH, J3 NC3FAH2-0, J4 NC3FAH2-0, J5 Conn_02x05_Odd_Even, Q1 IRF9540N, Q2 IRF9540N, U5 SC18IS606PWJ

Commit message: Update t-dsp_dual_preamp.kicad_pcb
Connections:
- IC1 pad 1: unconnected-(IC1-N/C_1-Pad1) -> Net-(IC1-N/C_1)
- IC1 pad 11: unconnected-(IC1-N/C_6-Pad11) -> Net-(IC1-N/C_1)
- IC1 pad 14: unconnected-(IC1-N/C_7-Pad14) -> Net-(IC1-N/C_1)
- IC1 pad 16: unconnected-(IC1-N/C_8-Pad16) -> Net-(IC1-N/C_1)
- IC1 pad 4: unconnected-(IC1-N/C_2-Pad4) -> Net-(IC1-N/C_1)
- IC1 pad 5: unconnected-(IC1-N/C_3-Pad5) -> Net-(IC1-N/C_1)
- IC1 pad 8: unconnected-(IC1-N/C_4-Pad8) -> Net-(IC1-N/C_1)
- IC1 pad 9: unconnected-(IC1-N/C_5-Pad9) -> Net-(IC1-N/C_1)
- IC2 pad 1: unconnected-(IC2-N/C_1-Pad1) -> Net-(IC2-N/C_1)
- IC2 pad 10: unconnected-(IC2-IN2-Pad10) -> GND
- IC2 pad 11: unconnected-(IC2-N/C_6-Pad11) -> Net-(IC2-N/C_1)
- IC2 pad 12: unconnected-(IC2-V-_1-Pad12) -> -15V
- IC2 pad 13: unconnected-(IC2-V+-Pad13) -> +15V
- IC2 pad 14: unconnected-(IC2-N/C_7-Pad14) -> Net-(IC2-N/C_1)
- IC2 pad 15: unconnected-(IC2-RG2-Pad15) -> Net-(IC2-RG2)
- IC2 pad 16: unconnected-(IC2-N/C_8-Pad16) -> Net-(IC2-N/C_1)
- IC2 pad 17: unconnected-(IC2-V-_2-Pad17) -> -15V
- IC2 pad 2: unconnected-(IC2-OUT2-Pad2) -> OUT-
- IC2 pad 3: unconnected-(IC2-OUT1-Pad3) -> OUT+
- IC2 pad 4: unconnected-(IC2-N/C_2-Pad4) -> Net-(IC2-N/C_1)
- IC2 pad 5: unconnected-(IC2-N/C_3-Pad5) -> Net-(IC2-N/C_1)
- IC2 pad 6: unconnected-(IC2-RG1-Pad6) -> Net-(IC2-RG1)
- IC2 pad 7: unconnected-(IC2-IN1-Pad7) -> Net-(D1-A)
- IC2 pad 8: unconnected-(IC2-N/C_4-Pad8) -> Net-(IC2-N/C_1)
- IC2 pad 9: unconnected-(IC2-N/C_5-Pad9) -> Net-(IC2-N/C_1)
- IC4 pad 1: unconnected-(IC4-SCAP2-Pad1) -> Net-(IC4-SCAP2)
- IC4 pad 10: unconnected-(IC4-TRC-Pad10) -> Net-(IC4-TRC)
- IC4 pad 11: unconnected-(IC4-VDD-Pad11) -> +3.3V
- IC4 pad 12: unconnected-(IC4-DGND-Pad12) -> GND
- IC4 pad 18: unconnected-(IC4-GPO3-Pad18) -> Net-(IC4-GPO3)
- IC4 pad 19: unconnected-(IC4-VEE-Pad19) -> -15V
- IC4 pad 2: unconnected-(IC4-RG1-Pad2) -> Net-(IC2-RG1)
- IC4 pad 20: unconnected-(IC4-VCC-Pad20) -> +15V
- IC4 pad 21: unconnected-(IC4-AGND-Pad21) -> GND
- IC4 pad 22: unconnected-(IC4-SOUT1-Pad22) -> Net-(IC4-SOUT1)
- IC4 pad 23: unconnected-(IC4-SOUT2-Pad23) -> Net-(IC4-SOUT2)
- IC4 pad 24: unconnected-(IC4-SCAP1-Pad24) -> Net-(IC4-SCAP1)
- IC4 pad 3: unconnected-(IC4-IN1-Pad3) -> OUT+
- IC4 pad 4: unconnected-(IC4-IN2-Pad4) -> OUT-
- IC4 pad 5: unconnected-(IC4-RG2-Pad5) -> Net-(IC2-RG2)
- IC4 pad 6: unconnected-(IC4-RST’-Pad6) -> RESET

Commit message: update
Parts:
- added C1: 22p, Capacitor_SMD:C_0805_2012Metric_Pad1.18x1.45mm_HandSolder, F.Cu at (-0.31, 157.5)
- added C10: 100p, Capacitor_SMD:C_0805_2012Metric_Pad1.18x1.45mm_HandSolder, F.Cu at (4.50, 163.5)
- added C11: 100p, Capacitor_SMD:C_0805_2012Metric_Pad1.18x1.45mm_HandSolder, F.Cu at (4.50, 166.5)
- added C12: 22u NP, Capacitor_SMD:C_0805_2012Metric_Pad1.18x1.45mm_HandSolder, F.Cu at (4.50, 169.5)
- added C13: 22u NP, Capacitor_SMD:C_0805_2012Metric_Pad1.18x1.45mm_HandSolder, F.Cu at (4.50, 172.5)
- added C14: 100N, Capacitor_SMD:C_0805_2012Metric_Pad1.18x1.45mm_HandSolder, F.Cu at (4.50, 175.5)
- added C15: 100N, Capacitor_SMD:C_0805_2012Metric_Pad1.18x1.45mm_HandSolder, F.Cu at (9.31, 157.5)
- added C16: 100N, Capacitor_SMD:C_0805_2012Metric_Pad1.18x1.45mm_HandSolder, F.Cu at (9.31, 160.5)
- added C2: 22p, Capacitor_SMD:C_0805_2012Metric_Pad1.18x1.45mm_HandSolder, F.Cu at (-0.31, 160.5)
- added C3: 220p, Capacitor_SMD:C_0805_2012Metric_Pad1.18x1.45mm_HandSolder, F.Cu at (-0.31, 163.5)
- added C4: 47u, Capacitor_SMD:C_0805_2012Metric_Pad1.18x1.45mm_HandSolder, F.Cu at (-0.31, 166.5)
- added C5: 47u, Capacitor_SMD:C_0805_2012Metric_Pad1.18x1.45mm_HandSolder, F.Cu at (-0.31, 169.5)
- added C6: 100p, Capacitor_SMD:C_0805_2012Metric_Pad1.18x1.45mm_HandSolder, F.Cu at (-0.31, 172.5)
- added C7: 100p, Capacitor_SMD:C_0805_2012Metric_Pad1.18x1.45mm_HandSolder, F.Cu at (-0.31, 175.5)
- added C8: 220p, Capacitor_SMD:C_0805_2012Metric_Pad1.18x1.45mm_HandSolder, F.Cu at (4.50, 157.5)
- added C9: 100n, Capacitor_SMD:C_0805_2012Metric_Pad1.18x1.45mm_HandSolder, F.Cu at (4.50, 160.5)
- added CT1: X, Capacitor_SMD:C_0805_2012Metric_Pad1.18x1.45mm_HandSolder, F.Cu at (9.31, 163.5)
- added D1: S1DB, Diode_SMD:D_SMA_Handsoldering, F.Cu at (16.8, 158.2)
- added D2: S1DB, Diode_SMD:D_SMA_Handsoldering, F.Cu at (16.8, 162.8)
- added D3: S1DB, Diode_SMD:D_SMA_Handsoldering, F.Cu at (16.8, 167.3)
- added D4: S1DB, Diode_SMD:D_SMA_Handsoldering, F.Cu at (16.8, 171.9)
- added R1: 1k2, Resistor_SMD:R_0805_2012Metric_Pad1.20x1.40mm_HandSolder, F.Cu at (-5.09, 157.4)
- added R18: 47K, Resistor_SMD:R_0805_2012Metric_Pad1.20x1.40mm_HandSolder, F.Cu at (-5.09, 181.1)
- added R2: 1k2, Resistor_SMD:R_0805_2012Metric_Pad1.20x1.40mm_HandSolder, F.Cu at (-5.09, 160.4)
- added R3: 10, Resistor_SMD:R_0805_2012Metric_Pad1.20x1.40mm_HandSolder, F.Cu at (-5.09, 163.3)
- added R4: 10, Resistor_SMD:R_0805_2012Metric_Pad1.20x1.40mm_HandSolder, F.Cu at (-5.09, 166.3)
- added R5: 6k81, Resistor_SMD:R_0805_2012Metric_Pad1.20x1.40mm_HandSolder, F.Cu at (-5.09, 169.2)
- added R6: 6k81, Resistor_SMD:R_0805_2012Metric_Pad1.20x1.40mm_HandSolder, F.Cu at (-5.09, 172.2)
- added R7: 1M2, Resistor_SMD:R_0805_2012Metric_Pad1.20x1.40mm_HandSolder, F.Cu at (-5.09, 175.2)
- added R8: 1M2, Resistor_SMD:R_0805_2012Metric_Pad1.20x1.40mm_HandSolder, F.Cu at (-5.09, 178.1)
- added RT1: X, Capacitor_SMD:C_0805_2012Metric_Pad1.18x1.45mm_HandSolder, F.Cu at (9.31, 166.5)
- added U1: PGA2505IDB, project_fp:PGA2505IDB, F.Cu at (105.0, 140.5)
- added board_outline3: board_outline, project_fp:audio_project_board_outline_100x70, F.Cu at (115.4, 84.9)
- board_outline2: footprint project_fp:audio_project_board_outline_100x70 -> project_fp:audio_project_board_outline_50x30
- moved J2 147.3 mm to (28.2, 40.4), turned to 180 degrees
- moved J1 147.2 mm to (28.2, 66.9), turned to 180 degrees
- moved J3 146.5 mm to (102.1, 34.9), turned to 0 degrees
- moved board_outline1 120.7 mm to (85.4, 17.2), turned to 180 degrees
- moved J4 96.4 mm to (102.1, 61.4), turned to 0 degrees
- moved U5 70.5 mm to (153.5, 174.0), turned to 180 degrees
- moved board_outline2 66.7 mm to (83.0, 179.5), turned to 0 degrees
- moved IC5 46.6 mm to (114.5, 161.5), turned to 180 degrees
- moved IC1 37.0 mm to (113.5, 171.0), turned to 180 degrees
- moved IC2 36.5 mm to (102.5, 171.2), turned to 180 degrees
- moved IC4 34.0 mm to (104.5, 162.0), turned to 180 degrees
- moved J5 31.0 mm to (126.7, 160.9), turned to 0 degrees
- moved Q2 23.3 mm to (87.0, 155.0), turned to -90 degrees
- moved Q1 12.0 mm to (87.5, 169.5), turned to -90 degrees

Commit message: update
Parts:
- removed C14: 100N, Capacitor_SMD:C_0805_2012Metric_Pad1.18x1.45mm_HandSolder
- removed CT1, RT1: X, Capacitor_SMD:C_0805_2012Metric_Pad1.18x1.45mm_HandSolder
- removed D1, D2, D3, D4: S1DB, Diode_SMD:D_SMA_Handsoldering
- removed IC1, IC2: 1583N16-U, project_fp:1583N16-U_QFN65P400X400X95-17N-D
- removed IC4, IC5: 5173N24-U, project_fp:5173N24-U_QFN65P500X500X95-25N-D
- removed Q1, Q2: IRF9540N, Package_TO_SOT_THT:TO-220-3_Vertical
- removed R1, R2: 1k2, Resistor_SMD:R_0805_2012Metric_Pad1.20x1.40mm_HandSolder
- removed R18: 47K, Resistor_SMD:R_0805_2012Metric_Pad1.20x1.40mm_HandSolder
- removed R3: 10, Resistor_SMD:R_0805_2012Metric_Pad1.20x1.40mm_HandSolder
- added C17: 4.7uF, Capacitor_SMD:C_1206_3216Metric_Pad1.33x1.80mm_HandSolder, F.Cu at (-40.0, 145.3)
- added C18: 4.7uF, Capacitor_SMD:C_1206_3216Metric_Pad1.33x1.80mm_HandSolder, F.Cu at (-26.0, 185.0)
- added C19: 47uF, Capacitor_SMD:CP_Elec_8x10.5, F.Cu at (-79.5, 170.5)
- added C20: 47uF, Capacitor_SMD:CP_Elec_8x10.5, F.Cu at (-79.5, 181.5)
- added C21: 1000pf, Capacitor_SMD:C_0805_2012Metric_Pad1.18x1.45mm_HandSolder, F.Cu at (-90.0, 169.0)
- added C22: 1000pf, Capacitor_SMD:C_0805_2012Metric_Pad1.18x1.45mm_HandSolder, F.Cu at (-90.0, 181.5)
- added C26: 4.7uF, Capacitor_SMD:C_1206_3216Metric_Pad1.33x1.80mm_HandSolder, F.Cu at (-25.0, 166.0)
- added C27: 4.7uF, Capacitor_SMD:C_1206_3216Metric_Pad1.33x1.80mm_HandSolder, F.Cu at (-25.0, 175.0)
- added CC1: 0, project_fp:R_0805_2012Metric_Pad1.20x1.40mm_HandSolder, F.Cu at (-51.5, 183.0)
- added CC2: 0, project_fp:R_0805_2012Metric_Pad1.20x1.40mm_HandSolder, F.Cu at (-48.5, 183.0)
- added D10: ~, Diode_SMD:D_SMA_Handsoldering, F.Cu at (-71.5, 170.5)
- added D11: S1DB, Diode_SMD:D_SMA_Handsoldering, F.Cu at (-71.5, 181.0)
- added D6: ~, Diode_SMD:D_SMA_Handsoldering, F.Cu at (-62.5, 170.5)
- added D7: ~, Diode_SMD:D_SMA_Handsoldering, F.Cu at (-67.0, 170.5)
- added D8: ~, Diode_SMD:D_SMA_Handsoldering, F.Cu at (-62.5, 181.0)
- added D9: ~, Diode_SMD:D_SMA_Handsoldering, F.Cu at (-67.0, 181.0)
- added J6: Conn_01x02, Connector_PinHeader_2.54mm:PinHeader_1x02_P2.54mm_Vertical, F.Cu at (-73.5, 143.0)
- added J8: 0, project_fp:R_0805_2012Metric_Pad1.20x1.40mm_HandSolder, F.Cu at (-51.5, 178.5)
- added J96: 0 ohm, project_fp:R_0805_2012Metric_Pad1.20x1.40mm_HandSolder, F.Cu at (-88.0, 143.9)
- added J97: 0 ohm, project_fp:R_0805_2012Metric_Pad1.20x1.40mm_HandSolder, F.Cu at (-88.0, 146.9)
- added J98: 0 ohm, project_fp:R_0805_2012Metric_Pad1.20x1.40mm_HandSolder, F.Cu at (-88.0, 149.8)
- added J99: 0 ohm, project_fp:R_0805_2012Metric_Pad1.20x1.40mm_HandSolder, F.Cu at (-88.0, 152.8)
- added JMP10: 0, project_fp:R_0805_2012Metric_Pad1.20x1.40mm_HandSolder, F.Cu at (-58.9, 152.0)
- added JMP11: 0, project_fp:R_0805_2012Metric_Pad1.20x1.40mm_HandSolder, F.Cu at (-58.6, 149.3)
- added R10: 0, project_fp:R_0805_2012Metric_Pad1.20x1.40mm_HandSolder, F.Cu at (-56.5, 183.0)
- added R10000: 10, project_fp:R_0805_2012Metric_Pad1.20x1.40mm_HandSolder, F.Cu at (-90.0, 166.5)
- added R100000: 10, project_fp:R_0805_2012Metric_Pad1.20x1.40mm_HandSolder, F.Cu at (-90.0, 184.0)
- added R11: 0, project_fp:R_0805_2012Metric_Pad1.20x1.40mm_HandSolder, F.Cu at (-56.5, 178.5)
- added R12: 0 ohm, project_fp:R_0805_2012Metric_Pad1.20x1.40mm_HandSolder, F.Cu at (-42.0, 185.0)
- added R13: 0 ohm, project_fp:R_0805_2012Metric_Pad1.20x1.40mm_HandSolder, F.Cu at (-39.5, 185.0)
- added R14: 0, project_fp:R_0805_2012Metric_Pad1.20x1.40mm_HandSolder, F.Cu at (-54.0, 183.0)
- added R15: 0, project_fp:R_0805_2012Metric_Pad1.20x1.40mm_HandSolder, F.Cu at (-48.5, 178.5)
- added R16: 6.81k, project_fp:R_0805_2012Metric_Pad1.20x1.40mm_HandSolder, F.Cu at (-90.0, 171.5)
- added R17: 6.81k, project_fp:R_0805_2012Metric_Pad1.20x1.40mm_HandSolder, F.Cu at (-90.0, 174.0)
- added R9: 10, project_fp:R_0805_2012Metric_Pad1.20x1.40mm_HandSolder, F.Cu at (-22.5, 175.0)
- C1, C2: value 22p -> 0.1uF
- C10: value 100p -> 1000pf
- C11, C6, C7: value 100p -> 0.1uF
- C12, C13: value 22u NP -> 0.1uF
- C15: value 100N -> 47uF; footprint Capacitor_SMD:C_0805_2012Metric_Pad1.18x1.45mm_HandSolder -> Capacitor_SMD:C_1206_3216Metric_Pad1.33x1.80mm_HandSolder
- C16: value 100N -> 4.7uF; footprint Capacitor_SMD:C_0805_2012Metric_Pad1.18x1.45mm_HandSolder -> Capacitor_SMD:C_1206_3216Metric_Pad1.33x1.80mm_HandSolder
- C3, C8: value 220p -> 0.1uF
- C4, C5: value 47u -> 0.1uF
- C9: value 100n -> 0.1uF
- J3, J4: value NC3FAH2-0 -> 0; footprint Connector_Audio:Jack_XLR_Neutrik_NC3FAH2-0_Horizontal -> project_fp:R_0805_2012Metric_Pad1.20x1.40mm_HandSolder
- R4: value 10 -> R_Small; footprint Resistor_SMD:R_0805_2012Metric_Pad1.20x1.40mm_HandSolder -> project_fp:R_0805_2012Metric_Pad1.20x1.40mm_HandSolder
- R5, R6: value 6k81 -> N/C; footprint Resistor_SMD:R_0805_2012Metric_Pad1.20x1.40mm_HandSolder -> project_fp:R_0805_2012Metric_Pad1.20x1.40mm_HandSolder
- R7, R8: value 1M2 -> 10; footprint Resistor_SMD:R_0805_2012Metric_Pad1.20x1.40mm_HandSolder -> project_fp:R_0805_2012Metric_Pad1.20x1.40mm_HandSolder
- moved board_outline1 253.7 mm to (-162.0, 73.3)
- moved J3 204.0 mm to (-35.0, 186.0), turned to 180 degrees
- moved J4 183.6 mm to (-35.0, 183.5), turned to 180 degrees
- moved U1 148.1 mm to (-39.0, 175.0), turned to -90 degrees
- moved C10 95.8 mm to (-90.0, 179.0)
- moved J5 90.1 mm to (180.4, 233.3)
- moved board_outline2 90.1 mm to (136.6, 251.9)
- moved R4 85.5 mm to (-90.0, 176.5), turned to 180 degrees
- moved C1 72.4 mm to (-72.0, 147.3)
- moved C15 60.9 mm to (-50.5, 145.8)
- moved U5 56.1 mm to (169.1, 227.9)
- moved R5 55.6 mm to (-59.0, 183.0), turned to -90 degrees
- moved R8 53.9 mm to (-59.0, 178.5), turned to 90 degrees
- moved R7 53.0 mm to (-58.0, 173.0), turned to -90 degrees
- moved C2 50.5 mm to (-50.0, 151.3)
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Connections:
- C1 pad 1: IN+ -> +48v
- C1 pad 2: ~ -> GNDPWR
- C10 pad 1: -15V -> Net-(C10-Pad1)
- C10 pad 2: GNDREF -> GNDPWR
- C11 pad 1: +15V -> Earth
- C11 pad 2: -15V -> -VA
- C12 pad 1: Net-(IC4-SOUT2) -> Earth
- C12 pad 2: Net-(IC4-SCAP2) -> -VA
- C13 pad 1: Net-(IC4-SOUT1) -> GND
- C13 pad 2: Net-(IC4-SCAP1) -> Net-(U1-VD-)
- C15 pad 1: +15V -> VCC
- C15 pad 2: unconnected-(C15-Pad2) -> GND
- C16 pad 1: +3.3V -> Earth
- C16 pad 2: GND -> -VA
- C2 pad 1: IN- -> VCC
- C2 pad 2: ~ -> GND
- C3 pad 1: IN+ -> Earth
- C3 pad 2: IN- -> GNDPWR
- C4 pad 1: IN+ -> Earth
- C4 pad 2: Net-(C4-Pad2) -> -VA
- C5 pad 1: IN- -> Earth
- C5 pad 2: Net-(C5-Pad2) -> +VA
- C6 pad 1: Net-(D1-A) -> Net-(U1-CS12)
- C6 pad 2: ~ -> Net-(U1-CS11)
- C7 pad 1: GND -> Net-(U1-CS22)
- C7 pad 2: ~ -> Net-(U1-CS21)
- C8 pad 1: Net-(D1-A) -> Earth
- C8 pad 2: GND -> Net-(J7-Pin_4)
- C9 pad 1: +15V -> Earth
- C9 pad 2: GNDREF -> +VA
- J3 pad 1: unconnected-(J3-Pad1) -> Net-(J7-Pin_4)
- J3 pad 2: unconnected-(J3-Pad2) -> Net-(U1-VCOMIN)
- J4 pad 1: unconnected-(J4-Pad1) -> Earth
- J4 pad 2: unconnected-(J4-Pad2) -> Net-(U1-VCOMIN)
- R4 pad 1: Net-(C5-Pad2) -> VIN1-
- R4 pad 2: GND -> VIO1+
- R5 pad 1: IN+ -> Net-(J8-Pad2)
- R5 pad 2: +48V -> Net-(R10-Pad2)
- R6 pad 1: IN- -> Net-(R11-Pad2)
- R6 pad 2: +48V -> Net-(J8-Pad2)
- R7 pad 1: GND -> Net-(C19-Pad2)
- R7 pad 2: Net-(IC4-SOUT2) -> Net-(D6-A)
- R8 pad 1: Net-(D1-A) -> Net-(C20-Pad2)
- R8 pad 2: Net-(IC4-SOUT1) -> Net-(D8-A)
- U1 pad 1: unconnected-(U1-AGND-Pad1) -> Earth
- U1 pad 10: unconnected-(U1-SCLK-Pad10) -> SCLK
- U1 pad 11: unconnected-(U1-SDO-Pad11) -> SDO
- U1 pad 12: unconnected-(U1-VD--Pad12) -> Net-(U1-VD-)
- U1 pad 13: unconnected-(U1-VA--Pad13) -> -VA
- U1 pad 14: unconnected-(U1-VOUT--Pad14) -> Net-(U1-VOUT-)
- U1 pad 15: unconnected-(U1-VOUT+-Pad15) -> Net-(U1-VOUT+)
- U1 pad 16: unconnected-(U1-VA+-Pad16) -> +VA
- U1 pad 17: unconnected-(U1-VA--Pad17) -> -VA
- U1 pad 18: unconnected-(U1-CS22-Pad18) -> Net-(U1-CS22)
- U1 pad 19: unconnected-(U1-CS21-Pad19) -> Net-(U1-CS21)
- U1 pad 2: unconnected-(U1-GPO1-Pad2) -> GPO1
- U1 pad 20: unconnected-(U1-CS12-Pad20) -> Net-(U1-CS12)
- U1 pad 21: unconnected-(U1-CS11-Pad21) -> Net-(U1-CS11)
- U1 pad 22: unconnected-(U1-VCOMIN-Pad22) -> Net-(U1-VCOMIN)
- U1 pad 23: unconnected-(U1-VIN--Pad23) -> Net-(U1-VIN-)
- U1 pad 24: unconnected-(U1-VIN+-Pad24) -> Net-(U1-VIN+)
- U1 pad 3: unconnected-(U1-GPO2-Pad3) -> GPO2
- U1 pad 4: unconnected-(U1-GPO3-Pad4) -> GPO3
- U1 pad 5: unconnected-(U1-GPO4-Pad5) -> GPO4
- U1 pad 6: unconnected-(U1-OVR-Pad6) -> OVR
- U1 pad 7: unconnected-(U1-DGND-Pad7) -> GND
- U1 pad 8: unconnected-(U1-SDI-Pad8) -> SDI
- U1 pad 9: unconnected-(U1-*CS-Pad9) -> CS

Commit message: update
Parts:
- removed C1, C11, C12, C13, C2, C3, C4, C5, C6, C7, C8, C9: 0.1uF, Capacitor_SMD:C_0805_2012Metric_Pad1.18x1.45mm_HandSolder
- removed C10, C21, C22: 1000pf, Capacitor_SMD:C_0805_2012Metric_Pad1.18x1.45mm_HandSolder
- removed C15: 47uF, Capacitor_SMD:C_1206_3216Metric_Pad1.33x1.80mm_HandSolder
- removed C16, C17, C18, C26, C27: 4.7uF, Capacitor_SMD:C_1206_3216Metric_Pad1.33x1.80mm_HandSolder
- removed C19, C20: 47uF, Capacitor_SMD:CP_Elec_8x10.5
- removed CC1, CC2, J3, J4, J8, JMP10, JMP11, R10, R11, R14, R15: 0, project_fp:R_0805_2012Metric_Pad1.20x1.40mm_HandSolder
- removed D10, D6, D7, D8, D9: ~, Diode_SMD:D_SMA_Handsoldering
- removed D11: S1DB, Diode_SMD:D_SMA_Handsoldering
- removed J5: Conn_02x05_Odd_Even, Connector_IDC:IDC-Header_2x05_P2.54mm_Vertical
- removed J6: Conn_01x02, Connector_PinHeader_2.54mm:PinHeader_1x02_P2.54mm_Vertical
- removed J96, J97, J98, J99, R12, R13: 0 ohm, project_fp:R_0805_2012Metric_Pad1.20x1.40mm_HandSolder
- removed R10000, R100000, R7, R8, R9: 10, project_fp:R_0805_2012Metric_Pad1.20x1.40mm_HandSolder
- removed R16, R17: 6.81k, project_fp:R_0805_2012Metric_Pad1.20x1.40mm_HandSolder
- removed R4: R_Small, project_fp:R_0805_2012Metric_Pad1.20x1.40mm_HandSolder
- removed R5, R6: N/C, project_fp:R_0805_2012Metric_Pad1.20x1.40mm_HandSolder
- removed U1: PGA2505IDB, project_fp:PGA2505IDB
- removed U5: SC18IS606PWJ, project_fp:SC18IS606PWJ_SOP65P640X110-16N
- removed board_outline2: board_outline, project_fp:audio_project_board_outline_50x30
- added J10: COMBO_NCJ6FA-H, project_fp:COMBO_XLR_NCJ6FI-H, F.Cu at (96.8, 111.8)
- added J9: COMBO_NCJ6FA-H, project_fp:COMBO_XLR_NCJ6FI-H, F.Cu at (96.3, 77.3)
- J1, J2: value XLRM_NC3FAH -> XLRM_NC3MAH; footprint project_fp:Jack_XLR_Neutrik_NC3FAH2_Horizontal -> project_fp:XLRM_NC3MAH
- board_outline3: footprint project_fp:audio_project_board_outline_100x70 -> project_fp:audio_project_board_outline_100x80
- moved board_outline1 309.8 mm to (145.2, 113.4), turned to 90 degrees
- moved J1 138.5 mm to (159.9, 109.8), turned to 90 degrees
- moved J2 136.3 mm to (160.0, 75.1), turned to 90 degrees
- moved board_outline3 76.3 mm to (177.8, 128.8)
Other:
- board size 100 x 70 mm -> 100 x 80 mm

Commit message: update
Parts:
- added C7: 470 uF Electrolytic Audio-Grade, project_fp:CP_Radial_D10.0mm_P5.00mm_AND_D8.0mm_P3.5mm, F.Cu at (114.1, 121.1)
- added C9: 470 uF Electrolytic Audio-Grade, project_fp:CP_Radial_D10.0mm_P5.00mm_AND_D8.0mm_P3.5mm, F.Cu at (115.6, 86.1)
- added J11: B2B-XH-A, project_fp:JST_B2B-XH-A, F.Cu at (105.0, 88.0)
- added J6: Conn_02x03_Odd_Even, project_fp:PREAMP_BYPASS_IDC-Header_2x03_P2.54mm_Vertical, F.Cu at (113.5, 109.8)
- added J7: Conn_02x03_Odd_Even, project_fp:PREAMP_BYPASS_IDC-Header_2x03_P2.54mm_Vertical, F.Cu at (113.5, 98.8)
- added J8: B2B-XH-A, project_fp:JST_B2B-XH-A, F.Cu at (105.0, 122.0)
- board_outline3: footprint project_fp:audio_project_board_outline_100x80 -> project_fp:audio_project_board_outline_100x50_minus2mounts
- moved J9 19.8 mm to (95.7, 97.1)
- moved J2 19.6 mm to (159.1, 94.7)
- moved board_outline1 12.8 mm to (152.7, 123.7)
- moved J1 10.9 mm to (159.1, 120.7)
- moved J10 9.87 mm to (95.7, 121.6)
- moved board_outline3 2.11 mm to (176.9, 126.9)
Connections:
- net /AUDIO_OUTP renamed /AUDIO_OUT1P
- board_outline1 pad 23: unconnected-(board_outline1-OUT1M-Pad23) -> /AUDIO_OUT1M
- board_outline1 pad 27: unconnected-(board_outline1-OUT2M-Pad27) -> /AUDIO_OUT2M
- board_outline1 pad 31: unconnected-(board_outline1-IN1M-Pad31) -> /AUDIO_IN1M
- board_outline1 pad 35: unconnected-(board_outline1-IN2M-Pad35) -> /AUDIO_IN2M
Other:
- board size 100 x 80 mm -> 100 x 50 mm

Commit message: update
Parts:
- board_outline3: footprint project_fp:audio_project_board_outline_100x50_minus2mounts -> project_fp:audio_project_board_outline_100x50_minus4mounts
- moved J10 60.3 mm to (100.0, 61.5), turned to 0 degrees
- moved J2 52.6 mm to (200.0, 61.5), turned to -90 degrees
- moved J1 52.0 mm to (200.0, 88.5), turned to -90 degrees
- moved C9 40.0 mm to (142.6, 56.6)
- moved J11 40.0 mm to (132.0, 58.5)
- moved J6 40.0 mm to (140.5, 80.3)
- moved J7 40.0 mm to (140.5, 69.3)
- moved J8 40.0 mm to (132.0, 92.5)
- moved board_outline1 40.0 mm to (179.7, 94.2)
- moved C7 40.0 mm to (141.1, 91.6)
- moved board_outline3 35.5 mm to (200.0, 100.0)
- moved J9 9.64 mm to (100.0, 88.5), turned to 0 degrees
