File: revisions/t-dsp_dual_preamp_PGA2505.kicad_sch (KiCad schematic)
At the start: 15 parts, among them J1 XLRM_NC3MAH, J10 COMBO_NCJ6FA-H, J2 XLRM_NC3MAH, J7 Conn_01x06, J9 COMBO_NCJ6FA-H, T108 Tab, T109 Tab, T110 Tab, T111 Tab

Commit message: update
Parts:
- added C1, C11, C12, C13, C2, C3, C4, C5, C6, C7, C8, C9: 0.1uF, Capacitor_SMD:C_0805_2012Metric_Pad1.18x1.45mm_HandSolder, symbol Device:C_Small
- added C10, C21, C22: 1000pf, Capacitor_SMD:C_0805_2012Metric_Pad1.18x1.45mm_HandSolder, symbol Device:C_Small
- added C15: 47uF, Capacitor_SMD:C_1206_3216Metric_Pad1.33x1.80mm_HandSolder, symbol Device:C_Polarized_Small
- added C16, C17, C18, C26, C27: 4.7uF, Capacitor_SMD:C_1206_3216Metric_Pad1.33x1.80mm_HandSolder, symbol Device:C_Polarized_Small
- added C19, C20: 47uF, Capacitor_SMD:CP_Elec_8x10.5, symbol Device:C_Polarized_Small
- added CC1, CC2: 0, project_fp:R_0805_2012Metric_Pad1.20x1.40mm_HandSolder, symbol Device:C_Small
- added D10, D6, D7, D8, D9: ~, Diode_SMD:D_SMA_Handsoldering, symbol Device:D_Small_Filled
- added D11: S1DB, Diode_SMD:D_SMA_Handsoldering, symbol Device:D_Small_Filled
- added J3, J4, J8, JMP10, JMP11, R10, R11, R14, R15: 0, project_fp:R_0805_2012Metric_Pad1.20x1.40mm_HandSolder, symbol Device:R_Small
- added J5: Conn_02x05_Odd_Even, Connector_IDC:IDC-Header_2x05_P2.54mm_Vertical, symbol Connector_Generic:Conn_02x05_Odd_Even
- added J6: Conn_01x02, Connector_PinHeader_2.54mm:PinHeader_1x02_P2.54mm_Vertical, symbol Connector_Generic:Conn_01x02
- added J96, J97, J98, J99: 0 ohm, project_fp:R_0805_2012Metric_Pad1.20x1.40mm_HandSolder, symbol Device:R
- added R10000, R100000, R7, R8, R9: 10, project_fp:R_0805_2012Metric_Pad1.20x1.40mm_HandSolder, symbol Device:R_Small
- added R12, R13: 0 ohm, project_fp:R_0805_2012Metric_Pad1.20x1.40mm_HandSolder, symbol Device:R_Small
- added R16, R17: 6.81k, project_fp:R_0805_2012Metric_Pad1.20x1.40mm_HandSolder, symbol Device:R_Small
- added R4: R_Small, project_fp:R_0805_2012Metric_Pad1.20x1.40mm_HandSolder, symbol Device:R_Small
- added R5, R6: N/C, project_fp:R_0805_2012Metric_Pad1.20x1.40mm_HandSolder, symbol Device:R_Small
- added U1: PGA2505IDB, DB24, symbol PGA2505IDB:PGA2505IDB
- added U5: SC18IS606PWJ, SC18IS606PWJ:SOP65P640X110-16N, symbol SC18IS606PWJ:SC18IS606PWJ
- added board_outline2: board_outline, project_fp:audio_project_board_outline_50x30, symbol project_lil_2:audio_project_board
- board_outline3: footprint project_fp:audio_project_board_outline_100x80 -> project_fp:audio_project_board_outline_100x70
Connections:
- net +12V: now also J5.1 (Pin_1), J5.3 (Pin_3)
- net +48V: now also J5.10 (Pin_10), J5.9 (Pin_9)
- net +48v: now also C1.1, J6.1 (Pin_1), R16.1, R17.2
- net +5VA: now also D10.1 (K), D6.1 (K), D8.1 (K)
- net +VA: now also C17.1, C26.1, C5.2, C9.2, U1.16 (VA+)
- net -12V: now also J5.5 (Pin_5), J5.7 (Pin_7)
- net -5VA: now also D11.2 (A), D7.2 (A), D9.2 (A)
- net -VA: now also C11.2, C12.2, C16.2, C27.2, C4.2, R9.1, U1.13 (VA-), U1.17 (VA-)
- net CS: now also U1.9 (*CS)
- net Earth: now also C11.1, C12.1, C16.1, C17.2, C26.2, C27.1, C3.1, C4.1, C5.1, C8.1, C9.1, D10.2 (A), D11.1 (K), J4.1, J8.1, JMP10.1, U1.1 (AGND)
- net G: now also J5.2 (Pin_2), J5.4 (Pin_4), J5.6 (Pin_6), J5.8 (Pin_8)
- net GND: now also C13.1, C15.2, C18.1, C2.2, J96.1, J97.1, J98.1, J99.1, JMP10.2, JMP11.2, U1.7 (DGND)
- net GNDPWR: now also C1.2, C10.2, C3.2, J6.2 (Pin_2)
- net GPO1: now also U1.2 (GPO1)
- net GPO2: now also U1.3 (GPO2)
- net GPO3: now also U1.4 (GPO3)
- net GPO4: now also U1.5 (GPO4)
- net OVR: now also U1.6 (OVR)
- net SCLK: now also U1.10 (SCLK)
- net SDI: now also U1.8 (SDI)
- net SDO: now also U1.11 (SDO)
- net SHIELD: now also JMP11.1
- net VCC: now also C15.1, C2.1
- net VIN1+: now also C21.2, R10000.1, R16.2, R4.2
- net VIN1-: now also C22.1, R100000.1, R17.1, R4.1
- net VOUT+: now also R12.1
- net VOUT-: now also R13.1
- net at J7.4 (Pin_4): now also C8.2, J3.1
- new net: R10.2, R14.1, R5.2
- new net: CC1.2, R14.2
- new net: J3.2, J4.2, U1.22 (VCOMIN)
- new net: J97.2, board_outline2.3 (GND)
- new net: D8.2 (A), D9.1 (K), R11.1, R8.2
- new net: R11.2, R15.2, R6.1
- new net: C13.2, C18.2, R9.2, U1.12 (VD-)
- new net: R13.2, U1.14 (VOUT-)
- new net: R12.2, U1.15 (VOUT+)
- new net: C7.1, U1.18 (CS22)
- new net: C7.2, U1.19 (CS21)
- new net: C6.1, U1.20 (CS12)
- new net: C6.2, U1.21 (CS11)
- new net: CC2.1, U1.23 (VIN-)
- new net: CC1.1, U1.24 (VIN+)
- new net: C10.1, C21.1, C22.2
- new net: J8.2, R5.1, R6.2
- new net: D6.2 (A), D7.1 (K), R10.1, R7.2
- new net: C20.1, R100000.2
- new net: C19.1, R10000.2
- new net: C19.2, R7.1
- new net: CC2.2, R15.1
- new net: C20.2, R8.1
- new net: J99.2, board_outline2.1 (GND)
- new net: J98.2, board_outline2.2 (GND)
- new net: J96.2, board_outline2.4 (GND)
